Commit message: Anchor SO-101 description to world link and remove ROS 1 transmissions

File: so101_description/urdf/so101_new_calib.urdf.xacro (robot description, xacro)
@@ -3,5 +3,6 @@
 <!-- Onshape https://cad.onshape.com/documents/7715cc284bb430fe6dab4ffd/w/4fd0791b683777b02f8d975a/e/826c553ede3b7592eb9ca800 -->
 <!-- Derived from so101_new_calib.urdf: adds wrist camera mount + wrist camera (Hex-Nut 32x32 UVC module form factor) -->
-<robot name="so101_new_calib">
+<!-- Source: https://github.com/TheRobotStudio/SO-ARM100, Simulation/SO101, commit 5f6d2b876a53a4872e405b991dd925556c9e38a4, Apache-2.0-->
+<robot xmlns:xacro="http://www.ros.org/wiki/xacro" name="so101_new_calib">
   <!-- Materials -->
   <material name="3d_printed">
@@ -11,4 +12,7 @@
     <color rgba="0.1 0.1 0.1 1.0"/>
   </material>
+  <!-- World Base -->
+  <link name="world">
+  </link>
   <!-- Link base -->
   <link name="base_link">
@@ -285,5 +289,4 @@
   <!-- Gripper frame (dummy link + fixed joint) -->
   <link name="gripper_frame_link">
-    <origin xyz="0 0 0" rpy="0 -0 0"/>
     <inertial>
       <origin xyz="0 0 0" rpy="0 0 0"/>
@@ -328,14 +331,4 @@
     <limit effort="10" velocity="10" lower="-0.174533" upper="1.74533"/>
   </joint>
-  <transmission name="gripper_trans">
-    <type>transmission_interface/SimpleTransmission</type>
-    <joint name="gripper">
-      <hardwareInterface>hardware_interface/PositionJointInterface</hardwareInterface>
-    </joint>
-    <actuator name="motor6">
-      <hardwareInterface>hardware_interface/PositionJointInterface</hardwareInterface>
-      <mechanicalReduction>1</mechanicalReduction>
-    </actuator>
-  </transmission>
   <!-- Joint from wrist to gripper -->
   <joint name="wrist_roll" type="revolute">
@@ -346,14 +339,4 @@
     <limit effort="10" velocity="10" lower="-2.74385" upper="2.84121"/>
   </joint>
-  <transmission name="wrist_roll_trans">
-    <type>transmission_interface/SimpleTransmission</type>
-    <joint name="wrist_roll">
-      <hardwareInterface>hardware_interface/PositionJointInterface</hardwareInterface>
-    </joint>
-    <actuator name="motor5">
-      <hardwareInterface>hardware_interface/PositionJointInterface</hardwareInterface>
-      <mechanicalReduction>1</mechanicalReduction>
-    </actuator>
-  </transmission>
   <!-- Joint from lower_arm to wrist -->
   <joint name="wrist_flex" type="revolute">
@@ -364,14 +347,4 @@
     <limit effort="10" velocity="10" lower="-1.65806" upper="1.65806"/>
   </joint>
-  <transmission name="wrist_flex_trans">
-    <type>transmission_interface/SimpleTransmission</type>
-    <joint name="wrist_flex">
-      <hardwareInterface>hardware_interface/PositionJointInterface</hardwareInterface>
-    </joint>
-    <actuator name="motor4">
-      <hardwareInterface>hardware_interface/PositionJointInterface</hardwareInterface>
-      <mechanicalReduction>1</mechanicalReduction>
-    </actuator>
-  </transmission>
   <!-- Joint from upper_arm to lower_arm -->
   <!-- Note: 5-degree calibration offset applied to joint limits -->
@@ -383,14 +356,4 @@
     <limit effort="10" velocity="10" lower="-1.69" upper="1.69"/>
   </joint>
-  <transmission name="elbow_flex_trans">
-    <type>transmission_interface/SimpleTransmission</type>
-    <joint name="elbow_flex">
-      <hardwareInterface>hardware_interface/PositionJointInterface</hardwareInterface>
-    </joint>
-    <actuator name="motor3">
-      <hardwareInterface>hardware_interface/PositionJointInterface</hardwareInterface>
-      <mechanicalReduction>1</mechanicalReduction>
-    </actuator>
-  </transmission>
   <!-- Joint from shoulder to upper_arm -->
   <joint name="shoulder_lift" type="revolute">
@@ -401,14 +364,4 @@
     <limit effort="10" velocity="10" lower="-1.74533" upper="1.74533"/>
   </joint>
-  <transmission name="shoulder_lift_trans">
-    <type>transmission_interface/SimpleTransmission</type>
-    <joint name="shoulder_lift">
-      <hardwareInterface>hardware_interface/PositionJointInterface</hardwareInterface>
-    </joint>
-    <actuator name="motor2">
-      <hardwareInterface>hardware_interface/PositionJointInterface</hardwareInterface>
-      <mechanicalReduction>1</mechanicalReduction>
-    </actuator>
-  </transmission>
   <!-- Joint from base to shoulder -->
   <joint name="shoulder_pan" type="revolute">
@@ -419,14 +372,10 @@
     <limit effort="10" velocity="10" lower="-1.91986" upper="1.91986"/>
   </joint>
-  <transmission name="shoulder_pan_trans">
-    <type>transmission_interface/SimpleTransmission</type>
-    <joint name="shoulder_pan">
-      <hardwareInterface>hardware_interface/PositionJointInterface</hardwareInterface>
-    </joint>
-    <actuator name="motor1">
-      <hardwareInterface>hardware_interface/PositionJointInterface</hardwareInterface>
-      <mechanicalReduction>1</mechanicalReduction>
-    </actuator>
-  </transmission>
+  <!-- Joint from world to base -->
+  <joint name="world_base_link" type="fixed">
+    <origin xyz = "0.0 0.0 0.0"/>
+    <parent link="world"/>
+    <child link="base_link"/>
+  </joint>
   <!-- Link wrist_camera_mount -->
   <link name="wrist_camera_mount_link">
