Commit message: so101_description: emit real-arm servo params via macro args
- Per-joint ID/sign/offset emitted only when hw == 'real' (so101_servo_params macro)
- baud_rate 1 Mbps, still to be confirmed against servo baud register
- Offsets are placeholders until the EEPROM table is recorded

File: so101_description/urdf/so101.ros2_control.xacro (robot description, xacro)
@@ -3,6 +3,13 @@
      only the hardware plugin changes with `hw`. -->
 <robot xmlns:xacro="http://www.ros.org/wiki/xacro">
+  <xacro:macro name="so101_servo_params" params="hw id sign offset">
+    <xacro:if value="${hw == 'real'}">
+      <param name="ID">${id}</param>
+      <param name="sign">${sign}</param>
+      <param name="offset">${offset}</param>
+    </xacro:if>
+  </xacro:macro>
   <!-- Arm joint: position command; position + velocity state -->
-  <xacro:macro name="so101_arm_joint" params="name">
+  <xacro:macro name="so101_arm_joint" params="name hw id sign offset">
     <joint name="${name}">
       <command_interface name="position"/>
@@ -11,4 +18,5 @@
       </state_interface>
       <state_interface name="velocity"/>
+      <xacro:so101_servo_params hw="${hw}" id="${id}" sign="${sign}" offset="${offset}"/>
     </joint>
   </xacro:macro>
@@ -29,11 +37,13 @@
                silently running something else. -->
           <plugin>so101_hardware/SO101System</plugin>
+          <param name="serial_port">/dev/ttyACM1</param>
+          <param name="baud_rate">1000000</param>
         </xacro:if>
       </hardware>
-      <xacro:so101_arm_joint name="shoulder_pan"/>
-      <xacro:so101_arm_joint name="shoulder_lift"/>
-      <xacro:so101_arm_joint name="elbow_flex"/>
-      <xacro:so101_arm_joint name="wrist_flex"/>
-      <xacro:so101_arm_joint name="wrist_roll"/>
+      <xacro:so101_arm_joint name="shoulder_pan"  hw="${hw}" id="1" sign="+1" offset="0"/>
+      <xacro:so101_arm_joint name="shoulder_lift" hw="${hw}" id="2" sign="+1" offset="0"/>
+      <xacro:so101_arm_joint name="elbow_flex"    hw="${hw}" id="3" sign="+1" offset="0"/>
+      <xacro:so101_arm_joint name="wrist_flex"    hw="${hw}" id="4" sign="+1" offset="0"/>
+      <xacro:so101_arm_joint name="wrist_roll"    hw="${hw}" id="5" sign="+1" offset="0"/>
       <!-- Gripper: position command; position + velocity + effort state.
            Effort is a load proxy, not calibrated torque (see README). -->
@@ -45,4 +55,5 @@
         <state_interface name="velocity"/>
         <state_interface name="effort"/>
+        <xacro:so101_servo_params hw="${hw}" id="6" sign="+1" offset="0"/>
       </joint>
     </ros2_control>

Commit message: so101_description: add expected EEPROM housing offsets for hw:=real

File: so101_description/urdf/so101.ros2_control.xacro (robot description, xacro)
@@ -3,13 +3,14 @@
      only the hardware plugin changes with `hw`. -->
 <robot xmlns:xacro="http://www.ros.org/wiki/xacro">
-  <xacro:macro name="so101_servo_params" params="hw id sign offset">
+  <xacro:macro name="so101_servo_params" params="hw id sign offset homing">
     <xacro:if value="${hw == 'real'}">
       <param name="ID">${id}</param>
       <param name="sign">${sign}</param>
       <param name="offset">${offset}</param>
+      <param name="eeprom_homing_offset">${homing}</param>
     </xacro:if>
   </xacro:macro>
   <!-- Arm joint: position command; position + velocity state -->
-  <xacro:macro name="so101_arm_joint" params="name hw id sign offset">
+  <xacro:macro name="so101_arm_joint" params="name hw id sign offset homing">
     <joint name="${name}">
       <command_interface name="position"/>
@@ -18,5 +19,5 @@
       </state_interface>
       <state_interface name="velocity"/>
-      <xacro:so101_servo_params hw="${hw}" id="${id}" sign="${sign}" offset="${offset}"/>
+      <xacro:so101_servo_params hw="${hw}" id="${id}" sign="${sign}" offset="${offset}" homing="${homing}"/>
     </joint>
   </xacro:macro>
@@ -33,7 +34,6 @@
         </xacro:if>
         <xacro:if value="${hw == 'real'}">
-          <!-- Implemented in M2. Until then this plugin does not exist, so the
-               controller manager fails loudly at load time instead of
-               silently running something else. -->
+          <!-- Real arm: STS3215 bus driver (so101_hardware). Configure is read-only on
+               the bus and fails if any servo's EEPROM disagrees with the params below. -->
           <plugin>so101_hardware/SO101System</plugin>
           <param name="serial_port">/dev/serial/by-id/usb-1a86_USB_Single_Serial_5AE6081270-if00</param>
@@ -41,9 +41,11 @@
         </xacro:if>
       </hardware>
-      <xacro:so101_arm_joint name="shoulder_pan"  hw="${hw}" id="1" sign="+1" offset="0"/>
-      <xacro:so101_arm_joint name="shoulder_lift" hw="${hw}" id="2" sign="+1" offset="0"/>
-      <xacro:so101_arm_joint name="elbow_flex"    hw="${hw}" id="3" sign="+1" offset="0"/>
-      <xacro:so101_arm_joint name="wrist_flex"    hw="${hw}" id="4" sign="+1" offset="0"/>
-      <xacro:so101_arm_joint name="wrist_roll"    hw="${hw}" id="5" sign="+1" offset="0"/>
+      <!-- eeprom_homing_offset: expected EEPROM Homing_Offset (counts), from LeRobot
+           follower calibration <file name>, <date>. Update after any LeRobot recalibration. -->
+      <xacro:so101_arm_joint name="shoulder_pan"  hw="${hw}" id="1" sign="+1" offset="0" homing="-2006"/>
+      <xacro:so101_arm_joint name="shoulder_lift" hw="${hw}" id="2" sign="+1" offset="0" homing="-1061"/>
+      <xacro:so101_arm_joint name="elbow_flex"    hw="${hw}" id="3" sign="+1" offset="0" homing="-1895"/>
+      <xacro:so101_arm_joint name="wrist_flex"    hw="${hw}" id="4" sign="+1" offset="0" homing="-1967"/>
+      <xacro:so101_arm_joint name="wrist_roll"    hw="${hw}" id="5" sign="+1" offset="0" homing="-2013"/>
       <!-- Gripper: position command; position + velocity + effort state.
            Effort is a load proxy, not calibrated torque (see README). -->
@@ -55,5 +57,5 @@
         <state_interface name="velocity"/>
         <state_interface name="effort"/>
-        <xacro:so101_servo_params hw="${hw}" id="6" sign="+1" offset="0"/>
+        <xacro:so101_servo_params hw="${hw}" id="6" sign="+1" offset="0" homing="1922"/>
       </joint>
     </ros2_control>

Commit message: so101_description: limits EEPROM ranges and measured wrist travel

File: so101_description/urdf/so101.ros2_control.xacro (robot description, xacro)
@@ -47,5 +47,5 @@
       <xacro:so101_arm_joint name="elbow_flex"    hw="${hw}" id="3" sign="+1" offset="0" homing="-1895"/>
       <xacro:so101_arm_joint name="wrist_flex"    hw="${hw}" id="4" sign="+1" offset="0" homing="-1967"/>
-      <xacro:so101_arm_joint name="wrist_roll"    hw="${hw}" id="5" sign="+1" offset="0" homing="-2013"/>
+      <xacro:so101_arm_joint name="wrist_roll" hw="${hw}" id="5" sign="+1" offset="0" homing="-2013" initial="-1.57"/>
       <!-- Gripper: position command; position + velocity + effort state.
            Effort is a load proxy, not calibrated torque (see README). -->
@@ -53,5 +53,5 @@
         <command_interface name="position"/>
         <state_interface name="position">
-          <param name="initial_value">0.0</param>
+          <param name="initial_value">${initial}</param>
         </state_interface>
         <state_interface name="velocity"/>

File: so101_description/urdf/so101_arm.xacro (robot description, xacro)
@@ -329,5 +329,5 @@
     <child link="moving_jaw_so101_v1_link"/>
     <axis xyz="0 0 1"/>
-    <limit effort="10" velocity="10" lower="-0.174533" upper="1.74533"/>
+    <limit effort="10" velocity="10" lower="-2.96" upper="-0.32"/>
   </joint>
   <!-- Joint from wrist to gripper -->
@@ -354,5 +354,5 @@
     <child link="lower_arm_link"/>
     <axis xyz="0 0 1"/>
-    <limit effort="10" velocity="10" lower="-1.69" upper="1.69"/>
+    <limit effort="10" velocity="10" lower="-1.69" upper="1.57"/>
   </joint>
   <!-- Joint from shoulder to upper_arm -->

Commit message: so101_description: correct <initial> tag placement in ros2_control.xacro

File: so101_description/urdf/so101.ros2_control.xacro (robot description, xacro)
@@ -12,9 +12,9 @@
   </xacro:macro>
   <!-- Arm joint: position command; position + velocity state -->
-  <xacro:macro name="so101_arm_joint" params="name hw id sign offset homing">
+  <xacro:macro name="so101_arm_joint" params="name hw id sign offset homing initial:=0.0">
     <joint name="${name}">
       <command_interface name="position"/>
       <state_interface name="position">
-        <param name="initial_value">0.0</param>
+        <param name="initial_value">${initial}</param>
       </state_interface>
       <state_interface name="velocity"/>
@@ -53,5 +53,4 @@
         <command_interface name="position"/>
         <state_interface name="position">
-          <param name="initial_value">${initial}</param>
         </state_interface>
         <state_interface name="velocity"/>
